File: production/pen-mixer.kicad_sch (KiCad schematic)
At the start: 31 parts, among them J1 USB-C 16P, J2 BAT, J3 FSR, U1 ISP1807-LR, U2 LSM6DS3TR-C, U3 MCP73831T-2ACI/OT, U4 TPS7A0533PDBV

Commit message: remake radio module
Claude-Session: https://claude.ai/code/session_01RCYT2QSY7BVZDeTyE9KrC4
Connections:
- net USB_DM: no longer J1.A6 (D+), J1.B6 (D+), U1.8 (D+)
- new net USB_DP: J1.A6 (D+), J1.B6 (D+), U1.8 (D+)

Commit message: add lcsc part numbers
Claude-Session: https://claude.ai/code/session_01RCYT2QSY7BVZDeTyE9KrC4
Parts:
- C1, C2: LCSC (none) -> C23733; MPN (none) -> CL05A475MP5NRNC; Manufacturer (none) -> Samsung Electro-Mechanics
- C10, C5, C7, C8, C9: LCSC (none) -> C1525; MPN (none) -> CL05B104KO5NNNC; Manufacturer (none) -> Samsung Electro-Mechanics
- C3, C4: LCSC (none) -> C52923; MPN (none) -> CL05A105KA5NQNC; Manufacturer (none) -> Samsung Electro-Mechanics
- C6: LCSC (none) -> C23692971; MPN (none) -> CGA0402X5R106M6R3GT; Manufacturer (none) -> TDK
- D1: LCSC (none) -> C130723; MPN (none) -> NCD0402G1; Manufacturer (none) -> Foshan NationStar
- J1: LCSC (none) -> C2988369; MPN (none) -> GT-USB-7010ASV; Manufacturer (none) -> G-Switch
- J2, J3: BOM Comments (none) -> bare solder pads - no part to order
- R1, R2: LCSC (none) -> C25905; MPN (none) -> 0402WGF5101TCE; Manufacturer (none) -> UNI-ROYAL
- R3: LCSC (none) -> C25765; MPN (none) -> 0402WGF2002TCE; Manufacturer (none) -> UNI-ROYAL
- R4: LCSC (none) -> C11702; MPN (none) -> 0402WGF1001TCE; Manufacturer (none) -> UNI-ROYAL
- R5: LCSC (none) -> C25744; MPN (none) -> 0402WGF1002TCE; Manufacturer (none) -> UNI-ROYAL
- R6, R7: LCSC (none) -> C25900; MPN (none) -> 0402WGF4701TCE; Manufacturer (none) -> UNI-ROYAL
- R8, R9: LCSC (none) -> C26083; MPN (none) -> 0402WGF1004TCE; Manufacturer (none) -> UNI-ROYAL
- TP1, TP2, TP4, TP5: BOM Comments (none) -> bare pad - no part
- U1: BOM Comments (none) -> 0 stock at JLC/LCSC - source from Mouser or DigiKey; LCSC (none) -> C5264268; MPN (none) -> ISP1807-LR-RS; Manufacturer (none) -> Insight SiP
- U2: LCSC (none) -> C967633; MPN (none) -> LSM6DS3TR-C; Manufacturer (none) -> STMicroelectronics
- U3: LCSC (none) -> C424093; MPN (none) -> MCP73831T-2ACI/OT; Manufacturer (none) -> Microchip
- U4: LCSC (none) -> C493453; MPN (none) -> TPS7A0533PDBVR; Manufacturer (none) -> Texas Instruments

Commit message: resize radio symbol body
Claude-Session: https://claude.ai/code/session_01RCYT2QSY7BVZDeTyE9KrC4
Parts:
- C1, C2: LCSC C23733 -> (none); MPN CL05A475MP5NRNC -> (none); Manufacturer Samsung Electro-Mechanics -> (none)
- C10, C5, C7, C8, C9: LCSC C1525 -> (none); MPN CL05B104KO5NNNC -> (none); Manufacturer Samsung Electro-Mechanics -> (none)
- C3, C4: LCSC C52923 -> (none); MPN CL05A105KA5NQNC -> (none); Manufacturer Samsung Electro-Mechanics -> (none)
- C6: LCSC C23692971 -> (none); MPN CGA0402X5R106M6R3GT -> (none); Manufacturer TDK -> (none)
- D1: LCSC C130723 -> (none); MPN NCD0402G1 -> (none); Manufacturer Foshan NationStar -> (none)
- J1: LCSC C2988369 -> (none); MPN GT-USB-7010ASV -> (none); Manufacturer G-Switch -> (none)
- J2, J3: BOM Comments bare solder pads - no part to order -> (none)
- R1, R2: LCSC C25905 -> (none); MPN 0402WGF5101TCE -> (none); Manufacturer UNI-ROYAL -> (none)
- R3: LCSC C25765 -> (none); MPN 0402WGF2002TCE -> (none); Manufacturer UNI-ROYAL -> (none)
- R4: LCSC C11702 -> (none); MPN 0402WGF1001TCE -> (none); Manufacturer UNI-ROYAL -> (none)
- R5: LCSC C25744 -> (none); MPN 0402WGF1002TCE -> (none); Manufacturer UNI-ROYAL -> (none)
- R6, R7: LCSC C25900 -> (none); MPN 0402WGF4701TCE -> (none); Manufacturer UNI-ROYAL -> (none)
- R8, R9: LCSC C26083 -> (none); MPN 0402WGF1004TCE -> (none); Manufacturer UNI-ROYAL -> (none)
- TP1, TP2, TP4, TP5: BOM Comments bare pad - no part -> (none)
- U1: BOM Comments 0 stock at JLC/LCSC - source from Mouser or DigiKey -> (none); LCSC C5264268 -> (none); MPN ISP1807-LR-RS -> (none); Manufacturer Insight SiP -> (none)
- U2: LCSC C967633 -> (none); MPN LSM6DS3TR-C -> (none); Manufacturer STMicroelectronics -> (none)
- U3: LCSC C424093 -> (none); MPN MCP73831T-2ACI/OT -> (none); Manufacturer Microchip -> (none)
- U4: LCSC C493453 -> (none); MPN TPS7A0533PDBVR -> (none); Manufacturer Texas Instruments -> (none)
Connections:
- net GND: no longer U2.2 (SDX)
- net USB_DM: no longer J1.B7 (D-)
- net USB_DP: no longer J1.B6 (D+)
- net VBAT: no longer U4.1 (IN)
- net VBAT_SENSE: no longer R8.2, R9.1
- new net: R8.2, R9.1
Other:
- moved on the sheet: C1, C10, C2, C3, C4, C5, C6, C7, C8, C9, D1, J1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
