File: production/v1/pen-mixer.kicad_sch (KiCad schematic)
At the start: 28 parts, among them J1 USB-C 16P, J2 BAT, U1 ISP1807-LR, U2 LSM6DS3TR-C, U3 MCP73831T-2ACI/OT, U4 TPS7A0533PDBV

Commit message: board v2 13x35
Claude-Session: https://claude.ai/code/session_01RCYT2QSY7BVZDeTyE9KrC4
Parts:
- J2: footprint pen-mixer:CONN-SMD_P2.00_S2B-PH-SM4-TB-LF-SN -> pen-mixer:SolderPad_1.2x2.0mm; BOM Comments mates JST PH 2.0 battery plug -> (none); LCSC C295747 -> (none); MPN S2B-PH-SM4-TB(LF)(SN) -> (none); Manufacturer JST -> (none)
Changed lines of the file:
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@@
 			)
 		)
-		(property "Footprint" "pen-mixer:CONN-SMD_P2.00_S2B-PH-SM4-TB-LF-SN"
+		(property "Footprint" "pen-mixer:SolderPad_1.2x2.0mm"
 			(at 74.93 92.71 0)
 			(hide yes)
@@
 			)
 		)
-		(property "BOM Comments" "mates JST PH 2.0 battery plug" (at 0 0 0)
-			(effects
-				(font
-					(size 1.27 1.27)
-				)
-				(hide yes)
-			)
-		)
-		(property "LCSC" "C295747" (at 0 0 0)
-			(effects
-				(font
-					(size 1.27 1.27)
-				)
-				(hide yes)
-			)
-		)
-		(property "Manufacturer" "JST" (at 0 0 0)
-			(effects
-				(font
-					(size 1.27 1.27)
-				)
-				(hide yes)
-			)
-		)
-		(property "MPN" "S2B-PH-SM4-TB(LF)(SN)" (at 0 0 0)
-			(effects
-				(font
-					(size 1.27 1.27)
-				)
-				(hide yes)
-			)
-		)
