File: production/kicad/pen-mixer.kicad_pcb (KiCad board)
At the start: 4 copper layers, 12.9 x 34.9 mm, 28 parts, among them J1 USB-C 16P, J2 BAT, U1 ISP1807-LR, U2 LSM6DS3TR-C, U3 MCP73831T-2ACI/OT, U4 TPS7A0533PDBV

Commit message: battery pads at tip
Claude-Session: https://claude.ai/code/session_01RCYT2QSY7BVZDeTyE9KrC4
Parts:
- J2: footprint CONN-SMD_P2.00_S2B-PH-SM4-TB-LF-SN -> SolderPad_1.2x2.0mm
- moved J2 2.93 mm to (102.2, 44.0)
Routing:
- net VBAT: track 48.3 -> 54.0 mm
- net GND: track 118.8 -> 119.8 mm
