File: production/kicad/pen-mixer.kicad_pcb (KiCad board)
At the start: 4 copper layers, 12.9 x 34.9 mm, 28 parts, among them J1 USB-C 16P, J2 BAT, U1 ISP1807-LR, U2 LSM6DS3TR-C, U3 MCP73831T-2ACI/OT, U4 TPS7A0533PDBV

Commit message: add v21 hardware
Claude-Session: https://claude.ai/code/session_01RCYT2QSY7BVZDeTyE9KrC4
Parts:
- added C11: 100n, C_0402_1005Metric, F.Cu at (107.4, 67.7)
- added LED1: XL-1010RGBC, LED-SMD_4P-L1.0-W1.0-TL_XL-1010RGBC-WS2812B, F.Cu at (107.6, 63.4)
- added LED2: XL-1010RGBC, LED-SMD_4P-L1.0-W1.0-TL_XL-1010RGBC-WS2812B, F.Cu at (107.6, 65.8)
- added SW1: EVQP7C01P, SW-SMD_EVQP7C01P, F.Cu at (107.0, 57.9)
- moved U4 1.70 mm to (102.9, 58.4)
- moved R4 1.00 mm to (105.7, 63.6)
- moved C1 0.70 mm to (105.0, 61.2)
- moved R9 0.30 mm to (105.9, 66.3)
Routing:
- net GND: track 119.8 -> 107.0 mm, vias 0 -> 4
- net +3V3: track 31.1 -> 36.0 mm
- net IMU_INT2: track 10.5 -> 15.4 mm
- net USB_DP: track 23.8 -> 26.5 mm
- net USB_DM: track 25.6 -> 23.2 mm
- net IMU_INT1: track 13.1 -> 15.2 mm
- net VBAT_SENSE: track 19.4 -> 17.6 mm
- net VBUS: track 42.1 -> 40.8 mm, vias 3 -> 5
- net SCL: track 23.5 -> 24.5 mm
- net LED_A: track 11.1 -> 12.1 mm
- net SDA: track 12.9 -> 11.9 mm
